File: cube/cube_4x4x4/cube_4x4x4.kicad_pcb (KiCad board)
At the start: 2 copper layers, 163 parts, among them P1 Column_0_0, P10 Column_4_4, P11 Column_0_5, P12 Column_4_5, P13 Column_0_6, P14 Column_4_6, P15 Column_0_7, P16 Column_4_7, P17 Column_1_0, P18 Column_5_0, P19 Column_1_1, P2 Column_4_0, P20 Column_5_1, P21 Column_1_2, P22 Column_5_2, P23 Column_1_3, P24 Column_5_3, P25 Column_1_4, P26 Column_5_4, P27 Column_1_5, P28 Column_5_5, P29 Column_1_6, P3 Column_0_1, P30 Column_5_6, P31 Column_1_7, P32 Column_5_7, P33 Column_2_0, P34 Column_6_0, P35 Column_2_1, P36 Column_6_1, P37 Column_2_2, P38 Column_6_2, P39 Column_2_3, P4 Column_4_1, P40 Column_6_3, P41 Column_2_4, P42 Column_6_4, P43 Column_2_5, P44 Column_6_5, P45 Column_2_6, P46 Column_6_6, P47 Column_2_7, P48 Column_6_7, P49 Column_3_0, P5 Column_0_2, P50 Column_7_0, P51 Column_3_1, P52 Column_7_1, P53 Column_3_2, P54 Column_7_2, P55 Column_3_3, P56 Column_7_3, P57 Column_3_4, P58 Column_7_4, P59 Column_3_5, P6 Column_4_2, P60 Column_7_5, P61 Column_3_6, P62 Column_7_6, P63 Column_3_7, P64 Column_7_7, P65 Layer 1, P66 Layer 2, P67 Layer 3, P68 Layer 5, P69 Layer 6, P7 Column_0_3, P70 Layer 7, P8 Column_4_3, P9 Column_0_4, Q1 BC337, Q2 BC337, Q3 BC337, Q4 BC337, Q5 BC337, Q6 BC337, Q7 BC337, Q8 BC337, U1 74HC595, U2 74HC595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

Commit message: cube kicad
Parts:
- moved U5 48.8 mm to (-70.6, 104.9)
- moved R17 18.6 mm to (-21.8, 58.9)
- moved R19 18.6 mm to (-8.89, 61.5)
- moved R21 18.6 mm to (-8.89, 58.9)
- moved R23 18.6 mm to (-8.89, 56.4)
- moved R25 18.6 mm to (-8.89, 53.8)
- moved R27 18.6 mm to (-8.89, 51.3)
- moved R29 18.6 mm to (-8.89, 48.8)
- moved R31 18.6 mm to (-8.89, 46.2)
- moved U3 18.6 mm to (-11.7, 61.5)
- moved U1 18.4 mm to (-11.7, 38.4)
- moved R11 18.4 mm to (-8.89, 28.2)
- moved R13 18.4 mm to (-8.89, 25.7)
- moved R15 18.4 mm to (-8.89, 23.1)
- moved R3 18.4 mm to (-8.89, 38.4)
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Routing:
- net Net-(P31-Pin_1): track 238.0 -> 0.00 mm
- net Net-(P15-Pin_1): track 238.0 -> 0.00 mm
- net Net-(P29-Pin_1): track 212.6 -> 0.00 mm
- net Net-(P13-Pin_1): track 212.6 -> 0.00 mm
- net Net-(P27-Pin_1): track 187.2 -> 0.00 mm
- net Net-(P11-Pin_1): track 187.2 -> 0.00 mm
- net Net-(P9-Pin_1): track 162.1 -> 0.00 mm
- net Net-(P25-Pin_1): track 161.8 -> 0.00 mm
- net Net-(P7-Pin_1): track 136.7 -> 0.00 mm
- net Net-(P23-Pin_1): track 136.4 -> 0.00 mm
- net Net-(P21-Pin_1): track 111.0 -> 0.00 mm
- net Net-(P5-Pin_1): track 111.0 -> 4.32 mm
- net Net-(P17-Pin_1): track 98.6 -> 0.00 mm
- net Net-(P1-Pin_1): track 98.4 -> 0.00 mm
- net Net-(P19-Pin_1): track 87.4 -> 1.78 mm
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