File: cube/cube_8x8x8/cube_8x8x8.kicad_pcb (KiCad board)
At the start: 2 copper layers, 164 parts, among them J1 Conn_01x02_Pin, P1 Column_0_0, P10 Column_4_4, P11 Column_0_5, P12 Column_4_5, P13 Column_0_6, P14 Column_4_6, P15 Column_0_7, P16 Column_4_7, P17 Column_1_0, P18 Column_5_0, P19 Column_1_1, P2 Column_4_0, P20 Column_5_1, P21 Column_1_2, P22 Column_5_2, P23 Column_1_3, P24 Column_5_3, P25 Column_1_4, P26 Column_5_4, P27 Column_1_5, P28 Column_5_5, P29 Column_1_6, P3 Column_0_1, P30 Column_5_6, P31 Column_1_7, P32 Column_5_7, P33 Column_2_0, P34 Column_6_0, P35 Column_2_1, P36 Column_6_1, P37 Column_2_2, P38 Column_6_2, P39 Column_2_3, P4 Column_4_1, P40 Column_6_3, P41 Column_2_4, P42 Column_6_4, P43 Column_2_5, P44 Column_6_5, P45 Column_2_6, P46 Column_6_6, P47 Column_2_7, P48 Column_6_7, P49 Column_3_0, P5 Column_0_2, P50 Column_7_0, P51 Column_3_1, P52 Column_7_1, P53 Column_3_2, P54 Column_7_2, P55 Column_3_3, P56 Column_7_3, P57 Column_3_4, P58 Column_7_4, P59 Column_3_5, P6 Column_4_2, P60 Column_7_5, P61 Column_3_6, P62 Column_7_6, P63 Column_3_7, P64 Column_7_7, P65 Layer 1, P66 Layer 2, P67 Layer 3, P68 Layer 5, P69 Layer 6, P7 Column_0_3, P70 Layer 7, P8 Column_4_3, P9 Column_0_4, Q1 BC337, Q2 BC337, Q3 BC337, Q4 BC337, Q5 BC337, Q6 BC337, Q7 BC337, Q8 BC337, U1 74HC595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

Commit message: cube kicad
Parts:
- moved Q8 379.4 mm to (-93.4, -6.00), turned to 180 degrees
- moved R72 368.5 mm to (-84.0, 15.4), turned to 90 degrees
- moved Q7 358.3 mm to (-82.4, -5.99), turned to 180 degrees
- moved R71 356.2 mm to (-81.6, 15.4), turned to 90 degrees
- moved Q6 352.9 mm to (-87.9, -5.99), turned to 180 degrees
- moved R70 345.0 mm to (-79.0, 15.4), turned to 90 degrees
- moved U9 338.6 mm to (-68.8, 18.7), turned to -90 degrees
- moved R69 335.1 mm to (-76.6, 15.4), turned to 90 degrees
- moved Q5 333.5 mm to (-76.9, -5.99), turned to 180 degrees
- moved R68 326.1 mm to (-73.9, 15.4), turned to 90 degrees
- moved Q4 320.2 mm to (-71.4, -5.99), turned to 180 degrees
- moved R67 318.6 mm to (-71.4, 15.4), turned to 90 degrees
- moved R66 312.7 mm to (-68.8, 15.4), turned to 90 degrees
- moved R65 308.6 mm to (-66.4, 15.4), turned to 90 degrees
- moved Q2 302.6 mm to (-66.0, -5.99), turned to 180 degrees
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Routing:
- net Net-(A1-D13): track 0.00 -> 168.3 mm, vias 0 -> 1
- net Net-(U1-SER): track 0.00 -> 79.3 mm
- net +VDC: track 0.00 -> 50.3 mm
- net Net-(U5-QH'): track 0.00 -> 42.3 mm
- net Net-(U3-QH'): track 0.00 -> 41.9 mm
- net Net-(U2-QH'): track 0.00 -> 41.6 mm
- net Net-(U4-QH'): track 0.00 -> 41.3 mm
- net Net-(U1-QH'): track 0.00 -> 40.9 mm
- net Net-(U6-QH'): track 0.00 -> 40.8 mm
- net Net-(U2-SER): track 0.00 -> 40.5 mm
- net -VDC: track 0.00 -> 34.1 mm
- net Net-(U3-QA): track 0.00 -> 15.5 mm
- net Net-(U1-QA): track 0.00 -> 15.4 mm
- net Net-(U1-QH): track 0.00 -> 2.62 mm
- net Net-(U1-QG): track 0.00 -> 2.62 mm
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